File: wiimote-ir-sensor.kicad_sch (KiCad schematic)
At the start: 10 parts, among them J1 Conn_01x04_Pin, U2 AP2112-3.3V, X1 X1G004451000300

Commit message: First usable revision
Parts:
- X1: value X1G004451000300 -> SG3225CAN 24.0000M-TJGA3; footprint Oscillator:Oscillator_SMD_SeikoEpson_SG8002LB-4Pin_5.0x3.2mm -> Oscillator:Oscillator_SMD_SeikoEpson_SG8002CE-4Pin_3.2x2.5mm_HandSoldering
Connections:
- net GND: no longer X1.1 (~{ST})
- no-connect marks 0 -> 1
Changed lines of the file:
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@@
   (junction (at 74.93 76.2) (diameter 0) (color 0 0 0 0)
   )
-  (junction (at 158.75 91.44) (diameter 0) (color 0 0 0 0)
-  )
   (junction (at 154.94 76.2) (diameter 0) (color 0 0 0 0)
   )
@@
   (junction (at 114.3 76.2) (diameter 0) (color 0 0 0 0)
   )
+  (no_connect (at 158.75 83.82))
   (wire (pts (xy 72.39 78.74) (xy 72.39 76.2))
     (stroke (width 0) (type default))
@@
     (stroke (width 0) (type default))
   )
-  (wire (pts (xy 154.94 91.44) (xy 158.75 91.44))
+  (wire (pts (xy 154.94 91.44) (xy 166.37 91.44))
     (stroke (width 0) (type default))
   )
@@
     (stroke (width 0) (type default))
   )
-  (wire (pts (xy 158.75 91.44) (xy 166.37 91.44))
-    (stroke (width 0) (type default))
-  )
   (wire (pts (xy 72.39 44.45) (xy 72.39 41.91))
     (stroke (width 0) (type default))
@@
   )
   (wire (pts (xy 182.88 83.82) (xy 182.88 125.73))
-    (stroke (width 0) (type default))
-  )
-  (wire (pts (xy 158.75 83.82) (xy 158.75 91.44))
     (stroke (width 0) (type default))
   )
@@
       (effects (font (size 1.27 1.27)))
     )
-    (property "Value" "X1G004451000300" (at 184.15 82.55 0)
-      (effects (font (size 1.27 1.27)))
-    )
-    (property "Footprint" "Oscillator:Oscillator_SMD_SeikoEpson_SG8002LB-4Pin_5.0x3.2mm" (at 184.15 92.71 0)
-      (effects (font (size 1.27 1.27)) hide)
-    )
+    (property "Value" "SG3225CAN 24.0000M-TJGA3" (at 184.15 82.55 0)
+      (effects (font (size 1.27 1.27)))
+    )
+    (property "Footprint" "Oscillator:Oscillator_SMD_SeikoEpson_SG8002CE-4Pin_3.2x2.5mm_HandSoldering" (at 184.15 92.71 0)
+      (effects (font (size 1.27 1.27)) hide)
+    )
