File: inline/wiimote-ir-sensor-inline.kicad_pcb (KiCad board)
At the start: 2 copper layers, 13 x 22.5 mm, 44 parts, among them J1 Conn_01x05_Pin, U2 AP2112-3.3V, X1 SG3225CAN 24.0000M-TJGA3

Commit message: Cheaper PCBA (#3)
* Move all components to one side of the board for cheaper PCBA

* Socketed: Add option to wire CLK directly
Parts:
- C1, C2, R1, U2: moved to F.Cu
- REF** (x32): footprint Panelization:NPTH-0.5mm -> wiimote-ir-sensor:NPTH-0.5mm
- X1: footprint Oscillator:Oscillator_SMD_SeikoEpson_SG8002CE-4Pin_3.2x2.5mm_HandSoldering -> Oscillator:Oscillator_SMD_SeikoEpson_SG8002CE-4Pin_3.2x2.5mm
- moved C3 5.98 mm to (105.1, 117.0), turned to 180 degrees
- moved C1 5.20 mm to (103.6, 112.3), turned to -90 degrees
- moved R2 4.74 mm to (107.9, 112.7)
- moved R1 3.76 mm to (105.3, 113.3), turned to -90 degrees
- moved JP1 3.07 mm to (109.0, 113.2), turned to 90 degrees
- moved X1 2.60 mm to (106.8, 109.3)
- moved U2 2.36 mm to (108.5, 115.7), turned to 90 degrees
- moved C2 1.99 mm to (109.5, 109.7), turned to 90 degrees
- moved R3 1.57 mm to (103.6, 108.8), turned to 90 degrees
Routing:
- net +3.3V: track 15.5 -> 10.8 mm, vias 4 -> 2
- net GND: track 11.1 -> 15.1 mm, vias 9 -> 7
- net VCC: track 10.6 -> 13.7 mm
- net /CLK: track 24.1 -> 22.6 mm, vias 2 -> 1
- net Net-(U1-RESET): track 6.32 -> 4.95 mm
- net /SCL: track 19.5 -> 18.3 mm
- net /SDA: track 17.9 -> 17.8 mm, vias 1 -> 2
- added copper zone on F.Cu, net +3.3V
- removed copper zone on B.Cu, net +3.3V
