File: inline/wiimote-ir-sensor-inline.kicad_sch (KiCad schematic)
At the start: 11 parts, among them J1 Conn_01x05_Pin, U2 AP2112-3.3V, X1 SG3225CAN 24.0000M-TJGA3

Commit message: Cheaper PCBA (#3)
* Move all components to one side of the board for cheaper PCBA

* Socketed: Add option to wire CLK directly
Parts:
- C2, C3: LCSC C519560 -> C15849
- J1: now not fitted; now left out of the parts list
- R1, R2: LCSC C114612 -> C13167
- R3: LCSC C126359 -> C4216
- U1: value ~ -> (none)
- X1: footprint Oscillator:Oscillator_SMD_SeikoEpson_SG8002CE-4Pin_3.2x2.5mm_HandSoldering -> Oscillator:Oscillator_SMD_SeikoEpson_SG8002CE-4Pin_3.2x2.5mm
